File: EMeterRMC.kicad_pcb (KiCad board)
At the start: 2 copper layers, 30 x 53 mm, 15 parts, among them J1 Conn_01x08, J2 Conn_01x09, Q1 IRLML6402, Q2 BCV62, SW1 BTN1, SW2 BTN3, SW3 BTN5, SW4 BTN2, SW5 BTN4, SW6 BTN6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

Commit message: corrected pcd
Parts:
- R1, R2: footprint Resistor_SMD:R_0805_2012Metric -> Resistor_SMD:R_0603_1608Metric
- SW1, SW2, SW3, SW4, SW5, SW6: footprint Button_Switch_SMD:SW_SPST_CK_KXT3 -> Button_Switch_SMD:SW_PCB_SNAPTRON_PNP-06
- moved SW4 10.5 mm to (121.2, 90.3)
- moved SW6 9.02 mm to (114.7, 106.8)
- moved SW1 9.00 mm to (107.9, 90.3)
- moved SW3 8.80 mm to (114.7, 97.4)
- moved SW5 8.66 mm to (124.0, 112.0)
- moved SW2 3.33 mm to (105.6, 111.8)
